Commit message: fix

File: assistive-gym-0.100/assistive_gym/envs/assets/laptop/laptop.urdf (robot description, URDF)
Before this commit: robot laptop.urdf, 2 links, 1 joints
Links:
- link baseLink: geometry collision box size=0.1 0.1 0.1; visual mesh filename=CursorControl/assistive-gym-0.100/assistive_gym/envs/assets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
- link screenLink: geometry collision box size=0.1 0.1 0.1; visual mesh filename=CursorControl/assistive-gym-0.100/assistive_gym/envs/assets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

Commit message: fix

File: assistive-gym-0.100/assistive_gym/envs/assets/laptop/laptop.urdf (robot description, URDF)
Before this commit: robot laptop.urdf, 2 links, 1 joints
Links:
- link baseLink: geometry collision box size=0.1 0.1 0.1; visual mesh filename=~/CursorControl/assistive-gym-0.100/assistive_gym/envs/asse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
- link screenLink: geometry collision box size=0.1 0.1 0.1; visual mesh filename=~/CursorControl/assistive-gym-0.100/assistive_gym/envs/asse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

Commit message: fix

File: assistive-gym-0.100/assistive_gym/envs/assets/laptop/laptop.urdf (robot description, URDF)
Before this commit: robot laptop.urdf, 2 links, 1 joints
Links:
- link baseLink: geometry collision box size=0.1 0.1 0.1; visual mesh filename=$(find edit_urdf)/CursorControl/assistive-gym-0.100/assisti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
- link screenLink: geometry collision box size=0.1 0.1 0.1; visual mesh filename=$(edit_urdf)/CursorControl/assistive-gym-0.100/assistive_gy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

Commit message: fix

File: assistive-gym-0.100/assistive_gym/envs/assets/laptop/laptop.urdf (robot description, URDF)
Before this commit: robot laptop.urdf, 2 links, 1 joints
Links:
- link screenLink: geometry collision box size=0.1 0.1 0.1; visual mesh filename=$(find edit_urdf)/CursorControl/assistive-gym-0.100/assisti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

Commit message: fix

File: assistive-gym-0.100/assistive_gym/envs/assets/laptop/laptop.urdf (robot description, URDF)
Before this commit: robot laptop.urdf, 2 links, 1 joints
Links:
- link baseLink: geometry collision box size=0.1 0.1 0.1; visual mesh filename=/home/schen/CursorControl/assistive-gym-0.100/assistive_gym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
- link screenLink: geometry collision box size=0.1 0.1 0.1; visual mesh filename=/home/schen/CursorControl/assistive-gym-0.100/assistive_gym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

Commit message: fix

File: assistive-gym-0.100/assistive_gym/envs/assets/laptop/laptop.urdf (robot description, URDF)
Before this commit: robot laptop.urdf, 2 links, 1 joints
Links:
- link baseLink: geometry collision box size=0.1 0.1 0.1; visual mesh filename=$(find urdf_tutorial)/CursorControl/assistive-gym-0.100/ass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
- link screenLink: geometry collision box size=0.1 0.1 0.1; visual mesh filename=$(find urdf_tutorial)/CursorControl/assistive-gym-0.100/ass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

Commit message: fix

File: assistive-gym-0.100/assistive_gym/envs/assets/laptop/laptop.urdf (robot description, URDF)
Before this commit: robot laptop.urdf, 2 links, 1 joints
Links:
- link baseLink: geometry collision box size=0.1 0.1 0.1; visual mesh filename=/home/schen/CursorControl/laptop/body_visual.obj
- link screenLink: geometry collision box size=0.1 0.1 0.1; visual mesh filename=/home/schen/CursorControl/laptop/screen_visual.obj
