Commit message: fix

File: laptop/laptop.urdf (robot description, URDF)
Before this commit: robot laptop.urdf, 2 links, 1 joints
Links:
- link baseLink: geometry collision box size=0.1 0.1 0.1; visual mesh filename=file:///home/schen/CursorControl/laptop/body_visual.obj
- link screenLink: geometry collision box size=0.1 0.1 0.1; visual mesh filename=file:///home/schen/CursorControl/laptop/screen_visual.obj

Commit message: fix

File: laptop/laptop.urdf (robot description, URDF)
Before this commit: robot laptop.urdf, 2 links, 1 joints
Links:
- removed link baseLink
- removed link screenLink
- added link base_link; collision box size=0.1 0.1 0.1; visual mesh filename=file:///home/schen/CursorControl/laptop/body_visual.obj
- added link screen_link; collision box size=0.1 0.1 0.1; visual mesh filename=file:///home/schen/CursorControl/laptop/screen_visual.obj
Joints:
- joint hinge: child screenLink -> screen_link; parent baseLink -> base_link

Commit message: fix

File: laptop/laptop.urdf (robot description, URDF)
Before this commit: robot laptop.urdf, 2 links, 1 joints
Links:
- link base_link: mass None -> .05
- link screen_link: mass None -> .01
