Commit message: deterministic encoder oneswitch model added

File: assistive-gym/assistive_gym/envs/assets/fridge/fridge.urdf (robot description, URDF)
Before this commit: robot oven.urdf, 5 links, 4 joints
Links:
- link base_link: geometry collision mesh filename=fridge.stl scale=1 1 1; visual mesh filename=fridge.stl scale=1 1 1
- link lower_door_link: geometry collision mesh filename=lower_door.stl scale=1 1 1; visual mesh filename=lower_door.stl scale=1 1 1
- link lower_handle_link: geometry collision mesh filename=lower_door_handle.stl scale=1 1 1; visual mesh filename=lower_door_handle.stl scale=1 1 1
- link upper_door_link: geometry collision mesh filename=upper_door.stl scale=1 1 1; visual mesh filename=upper_door.stl scale=1 1 1
- link upper_handle_link: geometry collision mesh filename=upper_door_handle.stl scale=1 1 1; visual mesh filename=upper_door_handle.stl scale=1 1 1
Joints:
- joint hinge: origin xyz=-.7 .6 1.4 rpy=0 0 0 -> xyz=-.55 .6 1.4 rpy=0 0 0

File: assistive-gym/assistive_gym/envs/assets/microwave/microwave.urdf (robot description, URDF)
Before this commit: robot microwave.urdf, 4 links, 3 joints
Joints:
- joint hinge: limit lower=-1.7 upper=0 effort=100 velocity=100 -> lower=-2.5 upper=0 effort=100 velocity=100
