Commit message: test -> master

File: assistive-gym/assistive_gym/envs/assets/bottle/bottle.urdf (robot description, URDF)
Before this commit: robot bottle.urdf, 1 links, 0 joints
Links:
- link baseLink: mass .0 -> None; geometry visual mesh filename=bottle.obj scale=2 2 1

File: assistive-gym/assistive_gym/envs/assets/shelf/shelf.urdf (robot description, URDF)
Before this commit: robot shelf.urdf, 1 links, 0 joints
Links:
- link baseLink: geometry collision box size=.02 .25 .42; collision box size=.02 .25 .42

Commit message: pretrain point reach

File: assistive-gym/assistive_gym/envs/assets/bottle/bottle.urdf (robot description, URDF)
Before this commit: robot bottle.urdf, 1 links, 0 joints
Links:
- link baseLink: mass None -> 0.01

Commit message: testing pretrain

File: assistive-gym/assistive_gym/envs/assets/bottle/bottle.urdf (robot description, URDF)
Before this commit: robot bottle.urdf, 1 links, 0 joints
Links:
- link baseLink: mass None -> .0
